Commit message: adjusted the model after testing against the robot

File: Model/panda_arm_hand.urdf (robot description, URDF)
Before this commit: robot panda_hand, 10 links, 9 joints
Joints:
- joint finger_joint1: origin xyz=0 0 0.1654 rpy=0 0 0 -> xyz=0 0 0.1654 rpy=0 0 -0.78539816339
- joint finger_joint2: axis 0 -1 0 -> 0 1 0; origin xyz=0 0 0.1654 rpy=0 0 0 -> xyz=0 0 0.1654 rpy=0 0 -0.78539816339
